Commit message: lab 4 teine tõmme

File: src/my_r2d2/urdf/r2d2.xacro (robot description, xacro)
@@ -233,3 +233,11 @@
     <origin xyz="0.04 0 0"/>
   </joint>
+  <link name="base_footprint">
+    <xacro:default_inertial mass="1"/>
+  </link>
+  <joint name="tofootprint" type="fixed">
+    <parent link="base_footprint"/>
+    <child link="base_link"/>
+    <origin xyz="0 0 0.47"/>
+  </joint>
 </robot>

Commit message: lab5

File: src/my_r2d2/urdf/r2d2.xacro (robot description, xacro)
@@ -241,3 +241,11 @@
     <origin xyz="0 0 0.47"/>
   </joint>
+  <link name="eye">
+    <xacro:default_inertial mass="1"/>
+  </link>
+  <joint name="toeye" type="fixed">
+    <parent link="lens"/>
+    <child link="eye"/>
+    <origin xyz="0.1 0 0" rpy="0 1.57075 0"/>
+  </joint>
 </robot>

Commit message: lab week 30

File: src/my_r2d2/urdf/r2d2.xacro (robot description, xacro)
@@ -242,10 +242,9 @@
   </joint>
   <link name="eye">
-    <xacro:default_inertial mass="1"/>
   </link>
   <joint name="toeye" type="fixed">
     <parent link="lens"/>
     <child link="eye"/>
-    <origin xyz="0.1 0 0" rpy="0 1.57075 0"/>
+    <origin xyz="-0.01 0 0" rpy="1.57075 3.1415 1.57075"/>
   </joint>
 </robot>
